Commit message: Added end-efector visualisation(works in sim)

File: src/robot_description/urdf/end_effector.urdf.xacro (robot description, xacro)
@@ -36,10 +36,11 @@
   <xacro:macro name="end_effector" params="prefix parent">
     <!-- Gripper link -->
-    <xacro:add_mesh_link name="${prefix}gripper" mesh_path="package://robot_description/meshes/RG2.stl"/>
+    <!-- <xacro:add_mesh_link name="${prefix}gripper" mesh_path="package://robot_description/meshes/RG2.stl"/> -->
+    <xacro:add_mesh_link name="${prefix}gripper" mesh_path="package://robot_description/meshes/Draft2.stl"/>
     <joint name="${prefix}gripper_joint" type="fixed">
       <parent link="${parent}"/>
       <child link="${prefix}gripper"/>
       <!-- <origin xyz="0 0 0.12" rpy="0 ${-pi/2} ${pi}"/> -->
-      <origin xyz="0 0.027 0.06" rpy="0 ${-pi/2} ${pi}"/>
+      <origin xyz="-0.025 0.025 0.06" rpy="${pi} 0 0"/>
     </joint>
   </xacro:macro>

Commit message: V1 Updated

File: src/robot_description/urdf/end_effector.urdf.xacro (robot description, xacro)
@@ -36,11 +36,10 @@
   <xacro:macro name="end_effector" params="prefix parent">
     <!-- Gripper link -->
-    <!-- <xacro:add_mesh_link name="${prefix}gripper" mesh_path="package://robot_description/meshes/RG2.stl"/> -->
-    <xacro:add_mesh_link name="${prefix}gripper" mesh_path="package://robot_description/meshes/Draft2.stl"/>
+    <xacro:add_mesh_link name="${prefix}gripper" mesh_path="package://robot_description/meshes/RG2.stl"/>
     <joint name="${prefix}gripper_joint" type="fixed">
       <parent link="${parent}"/>
       <child link="${prefix}gripper"/>
       <!-- <origin xyz="0 0 0.12" rpy="0 ${-pi/2} ${pi}"/> -->
-      <origin xyz="-0.025 0.025 0.06" rpy="${pi} 0 0"/>
+      <origin xyz="0 0.027 0.06" rpy="0 ${-pi/2} ${pi}"/>
     </joint>
   </xacro:macro>

Commit message: v1 Week11 Wed

File: src/robot_description/urdf/end_effector.urdf.xacro (robot description, xacro)
@@ -20,5 +20,6 @@
       <collision>
         <geometry>
-          <box size="0.05 0.1 0.1"/>
+          <!-- Temporarily disabled: set to minimal size for testing -->
+          <box size="0.001 0.001 0.001"/>
         </geometry>
         <origin xyz="0 0 0" rpy="0 0 0"/>
@@ -36,10 +37,11 @@
   <xacro:macro name="end_effector" params="prefix parent">
     <!-- Gripper link -->
-    <xacro:add_mesh_link name="${prefix}gripper" mesh_path="package://robot_description/meshes/RG2.stl"/>
+    <!-- <xacro:add_mesh_link name="${prefix}gripper" mesh_path="package://robot_description/meshes/RG2.stl"/> -->
+    <xacro:add_mesh_link name="${prefix}gripper" mesh_path="package://robot_description/meshes/wholedraft1.stl"/>
     <joint name="${prefix}gripper_joint" type="fixed">
       <parent link="${parent}"/>
       <child link="${prefix}gripper"/>
       <!-- <origin xyz="0 0 0.12" rpy="0 ${-pi/2} ${pi}"/> -->
-      <origin xyz="0 0.027 0.06" rpy="0 ${-pi/2} ${pi}"/>
+      <origin xyz="-0.025 0.04 0.104" rpy="${pi} 0 0"/>
     </joint>
   </xacro:macro>

File: src/robot_description/urdf/ur5e_with_camera.xacro (robot description, xacro)
@@ -15,5 +15,5 @@
   <xacro:arg name="camera_x" default="1.29163"/>
   <xacro:arg name="camera_y" default="0.0146956"/>
-  <xacro:arg name="camera_z" default="0.665489"/>
+  <xacro:arg name="camera_z" default="0.765489"/>
   <xacro:arg name="camera_roll"  default="0.0372615"/>
   <xacro:arg name="camera_pitch" default="-0.815369"/>
@@ -67,13 +67,14 @@
     trajectory_port="$(arg trajectory_port)"
     initial_positions="${dict(
-        shoulder_pan_joint=0.0,
-        shoulder_lift_joint=-1.57,
-        elbow_joint=0.0,
-        wrist_1_joint=0.0,
-        wrist_2_joint=0.0,
+        shoulder_pan_joint=3.14159,
+        shoulder_lift_joint=-1.5708,
+        elbow_joint=-1.5708,
+        wrist_1_joint=-1.5708,
+        wrist_2_joint=1.5708,
         wrist_3_joint=0.0)}"
   >
     <origin xyz="0 0 0" rpy="0 0 0"/>
   </xacro:ur_robot>
+  <!-- Home position: ros2 launch arm_manipulation move_arm_to_pose_launch.py x:=0.492 y:=0.133 z:=0.488 -->
   <!-- =========================================================
        Hand-eye camera definition
@@ -107,8 +108,10 @@
   <link name="camera_color_optical_frame"/>
   <!-- Transform from camera_link to camera_color_optical_frame -->
+  <!-- RealSense optical frame: rotate -90° around X, then -90° around Z -->
+  <!-- Quaternion (0.5, -0.5, 0.5, 0.5) = RPY (-π/2, 0, -π/2) -->
   <joint name="camera_color_optical_joint" type="fixed">
     <parent link="camera_link"/>
     <child link="camera_color_optical_frame"/>
-    <origin xyz="0 0 0" rpy="0 0 0"/>
+    <origin xyz="0 0 0" rpy="-1.5708 0 -1.5708"/>
   </joint>
   <!-- =========================================================

Commit message: Created README.md

File: src/robot_description/urdf/end_effector.urdf.xacro (robot description, xacro)
@@ -22,6 +22,7 @@
           <!-- Temporarily disabled: set to minimal size for testing -->
           <box size="0.001 0.001 0.001"/>
+          <!-- <box size="0.1 0.1 0.1"/>  -->
         </geometry>
-        <origin xyz="0 0 0" rpy="0 0 0"/>
+        <origin xyz="0 0 0.1" rpy="0 0 0"/>
       </collision>
       <inertial>
@@ -42,6 +43,6 @@
       <parent link="${parent}"/>
       <child link="${prefix}gripper"/>
-      <!-- <origin xyz="0 0 0.12" rpy="0 ${-pi/2} ${pi}"/> -->
-      <origin xyz="-0.025 0.04 0.104" rpy="${pi} 0 0"/>
+      <!-- <origin xyz="-0.025 0.04 0.104" rpy="${pi} 0 0"/> -->
+      <origin xyz="-0.0125 0.04 0.104" rpy="${pi} 0 0"/>
     </joint>
   </xacro:macro>
